File: schematics/Flip-dot_part.sch (KiCad schematic (older format))
At the start: 38 parts, among them U1 74HC85, U10 74HC238, U11 ULN2803A, U12 TBD62783A, U13 ULN2803A, U14 TBD62783A, U15 ULN2803A, U16 TBD62783A, U17 ULN2803A, U18 TBD62783A, U2 74HC238, U3 74HC238, U4 74HC238, U5 74HC238, U6 74HC238, U7 74HC238, U8 74HC238, U9 74HC238

Commit message: BAV99 fix
Parts:
- removed unit 2 of D1
- removed unit 2 of D2
- removed D3, D4, D7, D8: BAV99, Package_TO_SOT_SMD:SOT-23, symbol Diode:BAV99
- removed unit 2 of D5
- removed unit 2 of D6
- added D13, D14, D17, D18: BAV99, Package_TO_SOT_SMD:SOT-23, symbol Diode:BAV99
- renumbered D1 to D11, D2 to D12, D5 to D15, D6 to D16
Connections:
- wire segments 334 -> 322
Other:
- moved on the sheet: D11, D12, D15, D16, L1, L2, L5, L6
